File: I2C-dac.kicad_pcb (KiCad board)
At the start: 2 copper layers, 40 x 30 mm, 13 parts, among them J2 Conn_01x06, U1 MCP4725

Commit message: update,
Parts:
- J2: footprint Connector_PinHeader_2.54mm:PinHeader_1x06_P2.54mm_Vertical -> footprint-lib:Pin_Header_Straight_1x06_Pitch2.54mm
Routing:
- net /SDA: track 15.9 -> 18.4 mm
- net GND: track 42.2 -> 44.7 mm, vias 5 -> 4
